Commit message: Add XACRO properties

File: catkin_ws/src/hachiroku_bot/urdf/hachiroku_bot.xacro (robot description, xacro)
@@ -1,8 +1,11 @@
 <?xml version="1.0"?>
 <robot name="hachiroku_bot" xmlns:xacro="http://ros.org/wiki/xacro">
+    <xacro:property name="base_length"  value="1"/>
+    <xacro:property name="base_width"   value="1"/>
+    <xacro:property name="base_height"  value="1"/>
     <link name="base_link">
         <visual>
             <geometry>
-                <box size="1 1 1"/>
+                <box size="${base_length} ${base_width} ${base_height}"/>
             </geometry>
             <origin xyz="0 0 0.1"/>

Commit message: Add wheel macro, properties, definition

File: catkin_ws/src/hachiroku_bot/urdf/hachiroku_bot.xacro (robot description, xacro)
@@ -4,4 +4,23 @@
     <xacro:property name="base_width"   value="1"/>
     <xacro:property name="base_height"  value="1"/>
+    <xacro:property name="wheel_radius" value="0.05"/>
+    <xacro:property name="wheel_length" value="0.02"/>
+    <xacro:macro name="wheel" params="name x y z">
+    <link name="${name}">
+      <visual>
+        <geometry>
+          <cylinder radius="${wheel_radius}" length="${wheel_length}"/>
+        </geometry>
+        <origin xyz="${x} ${y} ${z}" rpy="1.5708 0 0"/>
+        <material name="black"/>
+      </visual>
+    </link>
+    <joint name="${name}_joint" type="continuous">
+      <parent link="base_link"/>
+      <child link="${name}"/>
+      <origin xyz="${x} ${y} ${z}" rpy="0 0 0"/>
+      <axis xyz="0 1 0"/>
+    </joint>
+  </xacro:macro>
     <link name="base_link">
         <visual>
@@ -12,3 +31,7 @@
         </visual>
     </link>
+    <xacro:wheel name="front_left_wheel" x="0.3" y="0.2" z="0.1"/>
+    <xacro:wheel name="front_right_wheel" x="0.3" y="-0.2" z="0.1"/>
+    <xacro:wheel name="rear_left_wheel" x="-0.3" y="0.2" z="0.1"/>
+    <xacro:wheel name="rear_right_wheel" x="-0.3" y="-0.2" z="0.1"/>
 </robot>

Commit message: Add color definition and modify values

File: catkin_ws/src/hachiroku_bot/urdf/hachiroku_bot.xacro (robot description, xacro)
@@ -1,10 +1,13 @@
 <?xml version="1.0"?>
 <robot name="hachiroku_bot" xmlns:xacro="http://ros.org/wiki/xacro">
-    <xacro:property name="base_length"  value="1"/>
-    <xacro:property name="base_width"   value="1"/>
-    <xacro:property name="base_height"  value="1"/>
+  <material name="black">
+    <color rgba="0 0 0 1"/>
+  </material>
     <xacro:property name="wheel_radius" value="0.05"/>
     <xacro:property name="wheel_length" value="0.02"/>
-    <xacro:macro name="wheel" params="name x y z">
+    <xacro:property name="base_length"  value="0.5"/>
+    <xacro:property name="base_width"   value="0.3"/>
+    <xacro:property name="base_height"  value="0.1"/>
+  <xacro:macro name="wheel" params="name x y z">
     <link name="${name}">
       <visual>
@@ -23,15 +26,15 @@
     </joint>
   </xacro:macro>
-    <link name="base_link">
-        <visual>
-            <geometry>
-                <box size="${base_length} ${base_width} ${base_height}"/>
-            </geometry>
-            <origin xyz="0 0 0.1"/>
-        </visual>
-    </link>
-    <xacro:wheel name="front_left_wheel" x="0.3" y="0.2" z="0.1"/>
-    <xacro:wheel name="front_right_wheel" x="0.3" y="-0.2" z="0.1"/>
-    <xacro:wheel name="rear_left_wheel" x="-0.3" y="0.2" z="0.1"/>
-    <xacro:wheel name="rear_right_wheel" x="-0.3" y="-0.2" z="0.1"/>
+  <link name="base_link">
+      <visual>
+          <geometry>
+              <box size="${base_length} ${base_width} ${base_height}"/>
+          </geometry>
+          <origin xyz="0 0 0.075"/>
+      </visual>
+  </link>
+  <xacro:wheel name="front_left_wheel" x="0.18" y="0.16" z="0.05"/>
+  <xacro:wheel name="front_right_wheel" x="0.18" y="-0.16" z="0.05"/>
+  <xacro:wheel name="rear_left_wheel" x="-0.18" y="0.16" z="0.05"/>
+  <xacro:wheel name="rear_right_wheel" x="-0.18" y="-0.16" z="0.05"/>
 </robot>

Commit message: Add black definition and LiDAR link

File: catkin_ws/src/hachiroku_bot/urdf/hachiroku_bot.xacro (robot description, xacro)
@@ -1,4 +1,7 @@
 <?xml version="1.0"?>
 <robot name="hachiroku_bot" xmlns:xacro="http://ros.org/wiki/xacro">
+  <material name="red">
+    <color rgba="1 0 0 1"/>
+  </material>
   <material name="black">
     <color rgba="0 0 0 1"/>
@@ -34,4 +37,18 @@
       </visual>
   </link>
+  <link name="lidar_link">
+      <visual>
+          <geometry>
+              <cylinder radius="0.03" length="0.028"/>
+          </geometry>
+          <origin xyz="0.2 0 0.128" rpy="0 0 1.5708"/>
+          <material name="red"/>
+      </visual>
+  </link>
+  <joint name="lidar_joint" type="fixed">
+      <parent link="base_link"/>
+      <child link="lidar_link"/>
+      <origin xyz="0 0 0.1" rpy="0 0 0"/>
+  </joint>
   <xacro:wheel name="front_left_wheel" x="0.18" y="0.16" z="0.05"/>
   <xacro:wheel name="front_right_wheel" x="0.18" y="-0.16" z="0.05"/>

Commit message: Add lidar property

File: catkin_ws/src/hachiroku_bot/urdf/hachiroku_bot.xacro (robot description, xacro)
@@ -12,4 +12,6 @@
     <xacro:property name="base_width"   value="0.3"/>
     <xacro:property name="base_height"  value="0.1"/>
+    <xacro:property name="lidar_height" value="0.028"/>
+    <xacro:property name="lidar_radius" value="0.03"/>
   <xacro:macro name="wheel" params="name x y z">
     <link name="${name}">
@@ -40,7 +42,7 @@
       <visual>
           <geometry>
-              <cylinder radius="0.03" length="0.028"/>
+              <cylinder radius="${lidar_radius}" length="${lidar_height}"/>
           </geometry>
-          <origin xyz="0.2 0 0.128" rpy="0 0 1.5708"/>
+          <origin xyz="0.2 0 0.128"/>
           <material name="red"/>
       </visual>

Commit message: Add collision and inertia for gazebo to render model

File: catkin_ws/src/hachiroku_bot/urdf/hachiroku_bot.xacro (robot description, xacro)
@@ -23,4 +23,14 @@
         <material name="black"/>
       </visual>
+      <collision>
+        <geometry>
+          <cylinder radius="${wheel_radius}" length="${wheel_length}"/>
+        </geometry>
+        <origin xyz="${x} ${y} ${z}" rpy="1.5708 0 0"/>
+      </collision>
+        <inertial>
+            <mass value="0.1"/>
+            <inertia ixx="0.001" iyy="0.001" izz="0.001" ixy="0" ixz="0" iyz="0"/>
+        </inertial>
     </link>
     <joint name="${name}_joint" type="continuous">
@@ -38,4 +48,14 @@
           <origin xyz="0 0 0.075"/>
       </visual>
+        <collision>
+            <geometry>
+                <box size="${base_length} ${base_width} ${base_height}"/>
+            </geometry>
+            <origin xyz="0 0 0.075"/>
+        </collision>
+        <inertial>
+            <mass value="1.0"/>
+            <inertia ixx="0.1" iyy="0.1" izz="0.1" ixy="0" ixz="0" iyz="0"/>
+        </inertial>
   </link>
   <link name="lidar_link">
@@ -47,4 +67,14 @@
           <material name="red"/>
       </visual>
+        <collision>
+            <geometry>
+                <cylinder radius="${lidar_radius}" length="${lidar_height}"/>
+            </geometry>
+            <origin xyz="0.2 0 0.128"/>
+        </collision>
+        <inertial>
+            <mass value="0.05"/>
+            <inertia ixx="0.001" iyy="0.001" izz="0.001" ixy="0" ixz="0" iyz="0"/>
+        </inertial>
   </link>
   <joint name="lidar_joint" type="fixed">

Commit message: Modify values to work for gazebo

File: catkin_ws/src/hachiroku_bot/urdf/hachiroku_bot.xacro (robot description, xacro)
@@ -20,5 +20,5 @@
           <cylinder radius="${wheel_radius}" length="${wheel_length}"/>
         </geometry>
-        <origin xyz="${x} ${y} ${z}" rpy="1.5708 0 0"/>
+        <origin xyz="0 0 0" rpy="1.5708 0 0"/>
         <material name="black"/>
       </visual>
@@ -27,5 +27,5 @@
           <cylinder radius="${wheel_radius}" length="${wheel_length}"/>
         </geometry>
-        <origin xyz="${x} ${y} ${z}" rpy="1.5708 0 0"/>
+        <origin xyz="0 0 0" rpy="1.5708 0 0"/>
       </collision>
         <inertial>
@@ -64,5 +64,5 @@
               <cylinder radius="${lidar_radius}" length="${lidar_height}"/>
           </geometry>
-          <origin xyz="0.2 0 0.128"/>
+          <origin xyz="0 0 0"/>
           <material name="red"/>
       </visual>
@@ -71,5 +71,5 @@
                 <cylinder radius="${lidar_radius}" length="${lidar_height}"/>
             </geometry>
-            <origin xyz="0.2 0 0.128"/>
+            <origin xyz="0 0 0"/>
         </collision>
         <inertial>
@@ -81,5 +81,5 @@
       <parent link="base_link"/>
       <child link="lidar_link"/>
-      <origin xyz="0 0 0.1" rpy="0 0 0"/>
+      <origin xyz="0.2 0 0.128" rpy="0 0 0"/>
   </joint>
   <xacro:wheel name="front_left_wheel" x="0.18" y="0.16" z="0.05"/>
